Commit message: Harden real-robot bringup: continuous voice, safer drive, Nav2 without docking.
Fix URDF launch YAML parse so the robot shows in RViz, keep a single cmd_vel path, stagger straight-drive PWM, and add voice room-matching tests.

File: src/hospital_description/urdf/robot.urdf (robot description, URDF)
Before this commit: robot custom_robo, 5 links, 4 joints
Links:
- link base_link: geometry collision box size=0.50 0.40 0.20; visual mesh filename=package://hospital_description/meshes/base.stl scale=0.001 0.001 0.001
- link laser: geometry collision cylinder length=0.04 radius=0.035; visual cylinder length=0.04 radius=0.035
- link left_wheel: geometry collision cylinder length=0.04 radius=0.0762; visual mesh filename=package://hospital_description/meshes/left_wheel.stl scale=0.001 0.001 0.001
- link right_wheel: geometry collision cylinder length=0.04 radius=0.0762; visual mesh filename=package://hospital_description/meshes/left_wheel.stl scale=0.001 0.001 0.001
Joints:
- joint base_footprint_to_base_link: origin xyz=0 0 0 rpy=0 0 0 -> xyz=0 0 0.0762 rpy=0 0 0
